File: bias_supply.sch (KiCad schematic (older format))
At the start: 16 parts, among them U401 TPS55340PWPR

Commit message: spun up integrated version
Parts:
- removed C401: 10u, Capacitors_SMD:C_0805_HandSoldering, symbol device:C
- removed C403, C405: 22n, Capacitors_SMD:C_0805_HandSoldering, symbol device:C
- removed C404: 510p, Capacitors_SMD:C_0805_HandSoldering, symbol device:C
- removed C406: 10u, Capacitors_SMD:CP_Elec_5x5.8, symbol device:CP
- removed C407: 680n, Capacitors_SMD:C_0805_HandSoldering, symbol device:C
- removed C408: 100n, Capacitors_SMD:C_0805_HandSoldering, symbol device:C
- removed D401: PDS760-13, DIO_PDS360-13:DIO_PDS360-13, symbol device:D_Schottky
- removed R401: 38k3, Resistors_SMD:R_0805_HandSoldering, symbol device:R
- removed R402: R, Resistors_SMD:R_0805_HandSoldering, symbol device:R
- removed U401: TPS55340PWPR, d4100_mod_board:SOP65P640X120-15N, symbol TPS55340PWPR:TPS55340PWPR
- added C301, C302, C304: 10u, Capacitors_SMD:C_1210_HandSoldering, symbol device:C
- added RV301: 1M, SamacSys_Parts:PVG5A502C03R00, symbol device:R_POT
- added TP301: BIAS_SW, Measurement_Points:Measurement_Point_Round-TH_Small, symbol conn:TEST_1P
- added TP302: BIAS_FB, Measurement_Points:Measurement_Point_Round-TH_Small, symbol conn:TEST_1P
- added TP303: VBIAS, Measurement_Points:Measurement_Point_Round-TH_Small, symbol conn:TEST_1P
- added TP304: GND, Measurement_Points:Measurement_Point_Square-TH_Small, symbol conn:TEST_1P
- added U301: TLV61046ADB, TO_SOT_Packages_SMD:SOT-23-6_Handsoldering, symbol Regulator_Switching:TLV61046ADB
- L301: renamed from L401; value 3u3 -> 15u; footprint XAL5030-332MEB:IND_XAL5030-332MEB -> SamacSys_Parts:WE-TPC_282892; symbol device:L_Core_Ferrite -> device:L; Vendor https://www.mouser.com/ProductDetail/Coilcraft/XAL5030-332M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 -> https://www.mouser.com/ProductDetail/Wurth-Elektronik/74402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
- R301: renamed from R403; value 210k -> 1M; Vendor (none) -> https://www.mouser.com/ProductDetail/Vishay-Dale/CRCW08051M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
- R302: renamed from R404; value 10k -> 71.5k; Vendor (none) -> https://www.mouser.com/ProductDetail/Vishay-Dale/CRCW080571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
- renumbered C402 to C303, NT402 to NT301
Connections:
- net Vin+: now also C301.1, C302.1; no longer C303.1
- net Vin-: now also C301.2, C302.2, C304.2, TP304.1, U301.2 (GND)
- net Vout+: now also C304.1, TP303.1, U301.5 (VOUT)
- net fb: now also RV301.2, TP302.1, U301.3 (FB); no longer R301.2
- net sw_loop: now also TP301.1, U301.1 (SW)
- net vin renamed boost_vin
- net boost_vin: now also C303.1, U301.4 (EN), U301.6 (VI)
- new net: R301.2, RV301.1
Other:
- moved on the sheet: C303, R301, R302
