File: d4100_mod_board_full.kicad_pcb (KiCad board)
At the start: 2 copper layers, 167.6 x 96.5 mm, 64 parts, among them J101 Conn_01x02, J102 Pogo_Pin, J103 Pogo_Pin, J104 Conn_01x02_Female, Q201 CSD18543Q3A, U201 LM25088MH-1, U401 TPS55340PWPR

Commit message: spun up integrated version
Parts:
- removed C212: 1u, Capacitors_SMD:C_0805_HandSoldering
- removed C213: 15u, Capacitors_SMD:C_2220_HandSoldering
- removed C214, C407: 680n, Capacitors_SMD:C_0805_HandSoldering
- removed C401: 10u, Capacitors_SMD:C_0805_HandSoldering
- removed C402, C408: 100n, Capacitors_SMD:C_0805_HandSoldering
- removed C403, C405: 22n, Capacitors_SMD:C_0805_HandSoldering
- removed C404: 510p, Capacitors_SMD:C_0805_HandSoldering
- removed C406: 10u, Capacitors_SMD:CP_Elec_5x5.8
- removed D201: SS3H10HE3_B/H, Diodes_SMD:D_SMC
- removed D401: PDS760-13, DIO_PDS360-13:DIO_PDS360-13
- removed L401: 3u3, XAL5030-332MEB:IND_XAL5030-332MEB
- removed NT201, NT204, NT206, NT402: Net-Tie_2, Oddities:NetTie-I_SMD
- removed NT202, NT203: Net-Tie_2, net_ties:NET-TIE-0.3mm
- removed Q201: CSD18543Q3A, CSD18543Q3A:SON65P300X315X90-9N
- removed R204: 4k75, Resistors_SMD:R_0805_HandSoldering
- removed R205: 10m, Resistors_SMD:R_0612
- removed R206: 36k5, Resistors_SMD:R_0805_HandSoldering
- removed R207: 3k4, Resistors_SMD:R_0805_HandSoldering
- removed R208: 35k7, Resistors_SMD:R_0805_HandSoldering
- removed R209: 1k65, Resistors_SMD:R_0805_HandSoldering
- removed R401: 38k3, Resistors_SMD:R_0805_HandSoldering
- removed R402: R, Resistors_SMD:R_0805_HandSoldering
- removed R403: 210k, Resistors_SMD:R_0805_HandSoldering
- removed R404: 10k, Resistors_SMD:R_0805_HandSoldering
- removed U401: TPS55340PWPR, TPS55340PWPR:SOP65P640X120-15N
- added C301: 10u, Capacitors_SMD:C_1210_HandSoldering, F.Cu at (98.5, 93.2)
- added C302: 10u, Capacitors_SMD:C_1210_HandSoldering, F.Cu at (95.2, 93.2)
- added C303: 100n, Capacitors_SMD:C_0805_HandSoldering, F.Cu at (92.4, 92.2)
- added C304: 10u, Capacitors_SMD:C_1210_HandSoldering, F.Cu at (86.9, 91.5)
- added J102a: Pogo_Pin, d4100_mod_board:mill-max_0985-x-15-20-71-14-11-0, F.Cu at (69.4, 123.4)
- added J103a: Pogo_Pin, d4100_mod_board:mill-max_0985-x-15-20-71-14-11-0, F.Cu at (94.2, 117.6)
- added L301: 15u, SamacSys_Parts:WE-TPC_282892, F.Cu at (96.1, 86.9)
- added NT301: Net-Tie_2, Oddities:NetTie-I_SMD, F.Cu at (92.3, 89.0)
- added R101: R, Resistors_SMD:R_0805_HandSoldering, F.Cu at (78.8, 126.5)
- added R102: R, Resistors_SMD:R_0805_HandSoldering, F.Cu at (101.0, 121.3)
- added R301: 1M, Resistors_SMD:R_0805_HandSoldering, F.Cu at (82.1, 89.6)
- added R302: 71.5k, Resistors_SMD:R_0805_HandSoldering, F.Cu at (87.9, 81.8)
- added RV201: R_POT, SamacSys_Parts:PVG5A502C03R00, F.Cu at (130.4, 107.1)
- added RV301: 1M, SamacSys_Parts:PVG5A502C03R00, F.Cu at (83.4, 82.9)
- added TP201: RESET_SW, Measurement_Points:Measurement_Point_Round-TH_Small, F.Cu at (148.5, 118.5)
- added TP202: RESET_FB, Measurement_Points:Measurement_Point_Round-TH_Small, F.Cu at (136.4, 107.2)
- added TP203: GND, Measurement_Points:Measurement_Point_Square-TH_Small, F.Cu at (141.6, 125.2)
- added TP204: VRESET, Measurement_Points:Measurement_Point_Round-TH_Small, F.Cu at (114.9, 116.8)
- added TP301: BIAS_SW, Measurement_Points:Measurement_Point_Round-TH_Small, F.Cu at (96.0, 82.4)
- added TP302: BIAS_FB, Measurement_Points:Measurement_Point_Round-TH_Small, F.Cu at (84.2, 77.1)
- added TP303: VBIAS, Measurement_Points:Measurement_Point_Round-TH_Small, F.Cu at (86.9, 96.7)
- added TP304: GND, Measurement_Points:Measurement_Point_Square-TH_Small, F.Cu at (90.8, 77.7)
- added U301: TLV61046ADB, TO_SOT_Packages_SMD:SOT-23-6_Handsoldering, F.Cu at (88.9, 87.2)
- C201: value 820n -> 22u; footprint Capacitors_SMD:C_0805_HandSoldering -> Capacitors_SMD:C_1210_HandSoldering
- C202: value 100n -> 22u; footprint Capacitors_SMD:C_0805_HandSoldering -> Capacitors_SMD:C_1210_HandSoldering
- C203: value 68n -> 4u7
- C204: value 22n -> 2u2
- C205: value 100n -> 470n
- C206: value 110p -> 4u7
- C207: value 47n -> 220p
- C208: value 100n -> 10u; footprint Capacitors_SMD:C_0805_HandSoldering -> Capacitors_SMD:C_1210_HandSoldering
- C209: value 14p -> 10u; footprint Capacitors_SMD:C_0805_HandSoldering -> Capacitors_SMD:C_1210_HandSoldering
- C210: value 150p -> 10u; footprint Capacitors_SMD:C_0805_HandSoldering -> Capacitors_SMD:C_1210_HandSoldering
- C211: value 130p -> 10u; footprint Capacitors_SMD:C_0805_HandSoldering -> Capacitors_SMD:C_1210_HandSoldering
- J101: moved to F.Cu
- L201: value 2u2 -> 33u; footprint d4100_mod_board:WE-LHMI_7030 -> SamacSys_Parts:SRN4012TA
- R201: value 10k -> R_Small
- R202: value 3k57 -> 39k
- R203: value 41k2 -> 1M
- U201: value LM25088MH-1 -> LM43601PWPR; footprint LM25088MH-1:SOP65P640X110-17N -> SamacSys_Parts:SOP65P640X120-17N
- moved R201 32.3 mm to (143.0, 112.6), turned to 90 degrees
- moved R202 28.6 mm to (135.4, 111.6), turned to 0 degrees
- moved C206 28.1 mm to (145.3, 112.7), turned to 90 degrees
- moved L201 23.4 mm to (141.2, 121.0), turned to 270 degrees
- moved R203 21.9 mm to (125.3, 106.8), turned to 90 degrees
- moved C204 18.9 mm to (147.4, 114.4), turned to 90 degrees
- moved J104 18.4 mm to (116.3, 88.6)
- moved C211 17.0 mm to (127.2, 121.9)
- moved C207 14.5 mm to (130.4, 111.6), turned to 0 degrees
- moved C203 14.4 mm to (124.6, 118.4)
- moved C208 13.2 mm to (130.4, 121.9), turned to 90 degrees
- moved C201 12.8 mm to (125.1, 112.7), turned to 90 degrees
- moved C205 12.7 mm to (144.9, 118.5), turned to 90 degrees
- moved U201 11.7 mm to (136.9, 115.5), turned to 180 degrees
- moved C210 11.0 mm to (137.0, 121.9), turned to 90 degrees
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Connections:
- C203 pad 1: /Reset Supply/enable -> +5V
- C204 pad 1: /Reset Supply/dither -> /Reset Supply/vcc
- C205 pad 1: /Reset Supply/vcc -> /Reset Supply/sw_loop
- C205 pad 2: /RESET+ -> /Reset Supply/boot
- C206 pad 1: /Reset Supply/ramp -> GND
- C207 pad 1: /Reset Supply/ss -> GND
- C207 pad 2: /RESET+ -> /Reset Supply/fb
- C208 pad 1: /Reset Supply/sw_loop -> GND
- C208 pad 2: /Reset Supply/bootstrap -> /RESET+
- C209 pad 1: /Reset Supply/fb -> GND
- C209 pad 2: /Reset Supply/comp -> /RESET+
- C210 pad 1: /Reset Supply/fb -> GND
- C210 pad 2: Net-(C210-Pad2) -> /RESET+
- C211 pad 1: /Reset Supply/fb -> GND
- C211 pad 2: Net-(C211-Pad2) -> /RESET+
- D101 pad 1: /bias_rail -> Net-(D101-Pad1)
- D102 pad 2: /reset_rail -> Net-(D102-Pad2)
- R201 pad 1: /Reset Supply/vin -> GND
- R201 pad 2: /Reset Supply/enable -> /Reset Supply/pgood
- R202 pad 1: /Reset Supply/enable -> /Reset Supply/fb
- R203 pad 1: /Reset Supply/vcc -> GND
- R203 pad 2: /Reset Supply/ramp -> Net-(R203-Pad2)
- U201 pad 1: /Reset Supply/vin -> /Reset Supply/sw_loop
- U201 pad 10: /Reset Supply/dither -> /RESET+
- U201 pad 11: /Reset Supply/sense- -> Net-(U201-Pad11)
- U201 pad 12: /Reset Supply/sense+ -> +5V
- U201 pad 13: /Reset Supply/sw_in -> +5V
- U201 pad 14: /Reset Supply/gate_drive -> +5V
- U201 pad 15: /Reset Supply/bootstrap -> /RESET+
- U201 pad 16: /Reset Supply/vcc -> /RESET+
- U201 pad 2: /Reset Supply/enable -> /Reset Supply/sw_loop
- U201 pad 3: /Reset Supply/ss -> /Reset Supply/boot
- U201 pad 4: /Reset Supply/ramp -> /Reset Supply/vcc
- U201 pad 5: /Reset Supply/rt -> GND
- U201 pad 6: /RESET+ -> Net-(U201-Pad6)
- U201 pad 7: /Reset Supply/comp -> Net-(U201-Pad7)
- U201 pad 8: /Reset Supply/fb -> /Reset Supply/pgood
- U201 pad 9: /Reset Supply/out_sense -> /Reset Supply/fb
Routing:
- net GND: track 10.2 -> 192.7 mm, vias 8 -> 28
- net /Reset Supply/vin: track 94.4 -> 0.00 mm
- net /Reset Supply/out_sense: track 79.8 -> 0.00 mm, vias 2 -> 0
- net +5V: track 13.7 -> 62.7 mm, vias 5 -> 0
- net /Reset Supply/fb: track 46.3 -> 12.6 mm, vias 2 -> 0
- net /Reset Supply/gate_drive: track 29.6 -> 0.00 mm
- net /BIAS+: track 36.9 -> 64.1 mm, vias 9 -> 0
- net /Reset Supply/vcc: track 29.4 -> 7.58 mm
- net /RESET+: track 18.0 -> 39.3 mm, vias 12 -> 8
- net /Reset Supply/enable: track 19.6 -> 0.00 mm
- net /Reset Supply/bootstrap: track 15.5 -> 0.00 mm
- net /Reset Supply/sense-: track 12.9 -> 0.00 mm, vias 2 -> 0
- net /Reset Supply/sense+: track 12.6 -> 0.00 mm, vias 2 -> 0
- net /Reset Supply/sw_loop: track 19.8 -> 11.1 mm, vias 3 -> 0
- net /Reset Supply/ramp: track 8.37 -> 0.00 mm
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- added copper zone on F.Cu, net /Bias Supply/boost_vin
- removed copper zone on B.Cu, net +5V
- removed copper zone on B.Cu, net /BIAS+
- removed copper zone on F.Cu, net /BIAS+
- removed copper zone on F.Cu, net /Bias Supply/sw_loop
- removed copper zone on F.Cu, net /Reset Supply/shunt+
- removed copper zone on B.Cu, net /Reset Supply/sw_loop
- removed copper zone on F.Cu, net /Reset Supply/sw_loop
- removed copper zone on F.Cu, net /Reset Supply/vin
Other:
- board size 167.6 x 96.5 mm -> 162.6 x 96.5 mm
- net class Power: clearance 0.381 -> 0.127
- board text added: "BIAS"
- board text added: "Continuity Check"
- board text added: "DLP Discovery D4100 Bias and Reset Mod Board Rev 2.0"
- board text added: "RESET"
