File: d4100_mod_board_full.sch (KiCad schematic (older format))
At the start: 16 parts, among them J101 Conn_01x02, J102 Pogo_Pin, J103 Pogo_Pin, J104 Conn_01x02_Female

Commit message: spun up integrated version
Parts:
- added R101, R102: R, Resistors_SMD:R_0805_HandSoldering, symbol device:R
Connections:
- net bias_rail: now also R101.1; no longer D101.1 (K)
- net reset_rail: now also R102.1; no longer D102.2 (A)
- new net: D101.1 (K), R101.2
- new net: D102.2 (A), R102.2
Other:
- moved on the sheet: C101, D101
Changed lines of the file:
@@
 Text Label 3700 4300 0    50   ~ 0
 reset_rail
-Wire Wire Line
-	5100 4700 5100 4300
 Connection ~ 5100 4300
 Wire Wire Line
@@
 Connection ~ 5100 5100
 $Comp
-L power:GND #PWR0104
+L power:GND #PWR0108
 U 1 1 5D0C0769
 P 8700 3350
-F 0 "#PWR0104" H 8700 3100 50  0001 C CNN
+F 0 "#PWR0108" H 8700 3100 50  0001 C CNN
 F 1 "GND" H 8705 3177 50  0000 C CNN
 F 2 "" H 8700 3350 50  0001 C CNN
@@
 	8700 3150 8750 3150
 $Comp
-L power:GND #PWR0110
+L power:GND #PWR0106
 U 1 1 5D0D5F8E
 P 8050 4800
-F 0 "#PWR0110" H 8050 4550 50  0001 C CNN
+F 0 "#PWR0106" H 8050 4550 50  0001 C CNN
 F 1 "GND" H 8055 4627 50  0000 C CNN
 F 2 "" H 8050 4800 50  0001 C CNN
@@
 	8050 4700 7900 4700
 $Comp
-L power:GND #PWR0108
+L power:GND #PWR0104
 U 1 1 5D0DB862
 P 7850 2900
-F 0 "#PWR0108" H 7850 2650 50  0001 C CNN
+F 0 "#PWR0104" H 7850 2650 50  0001 C CNN
 F 1 "GND" H 7855 2727 50  0000 C CNN
 F 2 "" H 7850 2900 50  0001 C CNN
@@
 	3450 4300 4700 4300
 $Comp
-L power:GND #PWR0106
+L power:GND #PWR0110
 U 1 1 5D1ABCFC
 P 9250 3850
-F 0 "#PWR0106" H 9250 3600 50  0001 C CNN
+F 0 "#PWR0110" H 9250 3600 50  0001 C CNN
 F 1 "GND" H 9255 3677 50  0000 C CNN
 F 2 "" H 9250 3850 50  0001 C CNN
@@
 	9250 3750 9300 3750
 $Comp
-L power:+5V #PWR0103
+L power:+5V #PWR0107
 U 1 1 5D1C9D26
 P 8700 3100
-F 0 "#PWR0103" H 8700 2950 50  0001 C CNN
+F 0 "#PWR0107" H 8700 2950 50  0001 C CNN
 F 1 "+5V" H 8715 3273 50  0000 C CNN
 F 2 "" H 8700 3100 50  0001 C CNN
@@
 	9250 3650 9300 3650
 $Comp
-L power:+5V #PWR0105
+L power:+5V #PWR0109
 U 1 1 5D1CD76D
 P 9250 3600
-F 0 "#PWR0105" H 9250 3450 50  0001 C CNN
+F 0 "#PWR0109" H 9250 3450 50  0001 C CNN
 F 1 "+5V" H 9265 3773 50  0000 C CNN
 F 2 "" H 9250 3600 50  0001 C CNN
@@
 	9250 3600 9250 3650
 $Comp
-L power:+5V #PWR0107
+L power:+5V #PWR0103
 U 1 1 5D1D3BF6
 P 7850 2600
-F 0 "#PWR0107" H 7850 2450 50  0001 C CNN
+F 0 "#PWR0103" H 7850 2450 50  0001 C CNN
 F 1 "+5V" H 7865 2773 50  0000 C CNN
 F 2 "" H 7850 2600 50  0001 C CNN
@@
 	7700 2650 7850 2650
 $Comp
-L power:+5V #PWR0109
+L power:+5V #PWR0105
 U 1 1 5D1D6377
 P 8050 4500
-F 0 "#PWR0109" H 8050 4350 50  0001 C CNN
+F 0 "#PWR0105" H 8050 4350 50  0001 C CNN
 F 1 "+5V" H 8065 4673 50  0000 C CNN
 F 2 "" H 8050 4500 50  0001 C CNN
@@
 Connection ~ 4700 2550
 Wire Wire Line
-	4700 2600 4700 2550
-Wire Wire Line
-	5100 2600 5100 2550
+	4700 2800 4700 2550
+Wire Wire Line
+	5100 3000 5100 2950
 $Comp
 L device:CP C101
 U 1 1 5D0930C4
-P 4700 2750
-F 0 "C101" H 4818 2796 50  0000 L CNN
-F 1 "4u7" H 4818 2705 50  0000 L CNN
-F 2 "Capacitors_Tantalum_SMD:CP_Tantalum_Case-C_EIA-6032-28_Reflow" H 4738 2600 50  0001 C CNN
-F 3 "https://www.mouser.com/datasheet/2/40/tps-776850.pdf" H 4700 2750 50  0001 C CNN
-F 4 "https://www.mouser.com/ProductDetail/AVX/TPSC475K035R0600?qs=%2Fha2pyFaduglChbUjLQpjYi93MlbS%2F0%2FZAO9XOBpQeTQ9QaxImqcQA%3D%3D" H 4700 2750 50  0001 C CNN "Vendor"
-	1    4700 2750
-	1    0    0    -1
-$EndComp
-Wire Wire Line
-	4700 3000 4700 2900
-Wire Wire Line
-	5100 3000 4700 3000
-Connection ~ 4700 3000
-Text Label 6000 3000 0    50   ~ 0
+P 4700 2950
+F 0 "C101" H 4818 2996 50  0000 L CNN
+F 1 "4u7" H 4818 2905 50  0000 L CNN
+F 2 "Capacitors_Tantalum_SMD:CP_Tantalum_Case-C_EIA-6032-28_Reflow" H 4738 2800 50  0001 C CNN
+F 3 "https://www.mouser.com/datasheet/2/40/tps-776850.pdf" H 4700 2950 50  0001 C CNN
+F 4 "https://www.mouser.com/ProductDetail/AVX/TPSC475K035R0600?qs=%2Fha2pyFaduglChbUjLQpjYi93MlbS%2F0%2FZAO9XOBpQeTQ9QaxImqcQA%3D%3D" H 4700 2950 50  0001 C CNN "Vendor"
+	1    4700 2950
+	1    0    0    -1
+$EndComp
+Wire Wire Line
+	4700 3400 4700 3100
+Wire Wire Line
+	5100 3400 4700 3400
+Connection ~ 4700 3400
+Text Label 6000 3400 0    50   ~ 0
 BIAS-
 $Comp
 L power:GND #PWR0101
 U 1 1 5D0A4D96
-P 4700 3050
-F 0 "#PWR0101" H 4700 2800 50  0001 C CNN
-F 1 "GND" H 4705 2877 50  0000 C CNN
-F 2 "" H 4700 3050 50  0001 C CNN
-F 3 "" H 4700 3050 50  0001 C CNN
-	1    4700 3050
-	1    0    0    -1
-$EndComp
-Wire Wire Line
-	4700 3050 4700 3000
-Wire Wire Line
-	5100 2900 5100 3000
-Connection ~ 5100 3000
+P 4700 3450
+F 0 "#PWR0101" H 4700 3200 50  0001 C CNN
+F 1 "GND" H 4705 3277 50  0000 C CNN
+F 2 "" H 4700 3450 50  0001 C CNN
+F 3 "" H 4700 3450 50  0001 C CNN
+	1    4700 3450
+	1    0    0    -1
+$EndComp
+Wire Wire Line
+	4700 3450 4700 3400
+Wire Wire Line
+	5100 3300 5100 3400
+Connection ~ 5100 3400
 $Comp
 L device:D_Zener D101
 U 1 1 5D09385A
-P 5100 2750
-F 0 "D101" V 5054 2829 50  0000 L CNN
-F 1 "BZV55B27" V 5145 2829 50  0000 L CNN
-F 2 "Diodes_SMD:D_MiniMELF" H 5100 2750 50  0001 C CNN
-F 3 "https://www.mouser.com/datasheet/2/395/BZV55B2V4_Series_F1804-1393200.pdf" H 5100 2750 50  0001 C CNN
-F 4 "https://www.mouser.com/ProductDetail/Taiwan-Semiconductor/BZV55B27-L1?qs=sGAEpiMZZMtQ8nqTKtFS%2FBBvJ4zpFTk1FiiiGr9sANE%3D" V 5100 2750 50  0001 C CNN "Vendor"
-	1    5100 2750
+P 5100 3150
+F 0 "D101" V 5054 3229 50  0000 L CNN
+F 1 "BZV55B27" V 5145 3229 50  0000 L CNN
+F 2 "Diodes_SMD:D_MiniMELF" H 5100 3150 50  0001 C CNN
+F 3 "https://www.mouser.com/datasheet/2/395/BZV55B2V4_Series_F1804-1393200.pdf" H 5100 3150 50  0001 C CNN
+F 4 "https://www.mouser.com/ProductDetail/Taiwan-Semiconductor/BZV55B27-L1?qs=sGAEpiMZZMtQ8nqTKtFS%2FBBvJ4zpFTk1FiiiGr9sANE%3D" V 5100 3150 50  0001 C CNN "Vendor"
+	1    5100 3150
 	0    1    1    0
 $EndComp
@@
 	5550 2550 6000 2550
 Wire Wire Line
-	5100 3000 6000 3000
+	5100 3400 6000 3400
+$Comp
+L device:R R101
+U 1 1 5D46EE39
+P 5100 2800
+F 0 "R101" H 5170 2846 50  0000 L CNN
+F 1 "R" H 5170 2755 50  0000 L CNN
+F 2 "Resistors_SMD:R_0805_HandSoldering" V 5030 2800 50  0001 C CNN
+F 3 "~" H 5100 2800 50  0001 C CNN
+	1    5100 2800
+	1    0    0    -1
+$EndComp
+Wire Wire Line
+	5100 2650 5100 2550
+$Comp
+L device:R R102
+U 1 1 5D46F51F
+P 5100 4500
+F 0 "R102" H 5170 4546 50  0000 L CNN
+F 1 "R" H 5170 4455 50  0000 L CNN
+F 2 "Resistors_SMD:R_0805_HandSoldering" V 5030 4500 50  0001 C CNN
+F 3 "~" H 5100 4500 50  0001 C CNN
+	1    5100 4500
+	1    0    0    -1
+$EndComp
+Wire Wire Line
+	5100 4350 5100 4300
+Wire Wire Line
+	5100 4650 5100 4700
 $EndSCHEMATC
